File: PrecisionTimer_RevF/PCB Design Files/PrecisionTimer_RevF.kicad_pcb (KiCad board)
At the start: 4 copper layers, 84.3 x 50.8 mm, 115 parts, among them J1 USB_B, J2 Micro_SD_Card, J3 1-1734775-1, J4 Barrel_Jack_Switch, J5 Conn_Coaxial, J6 Conn_02x05_Odd_Even, J7 Conn_Coaxial, J8 Conn_Coaxial, J9 Conn_01x04_Male, Q1 Q_NMOS_GSD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

Commit message: Add files via upload
Parts:
- moved C32 0.72 mm to (139.9, 69.4), turned to 90 degrees
- moved FB6 0.20 mm to (167.9, 68.0)
Routing:
- net UART_RX: track 40.4 -> 39.0 mm
- net RST: track 42.0 -> 43.3 mm
- net UART_TX: track 39.3 -> 38.1 mm
- net MCCDA: track 43.2 -> 42.6 mm
- net MCCK: track 43.5 -> 43.0 mm
Other:
- board text added: "MIPI10"
- board text removed: "MIPI-10"
