File: PrecisionTimer_RevG.1/PCB Design Files/PrecisionTimer_RevG-1.kicad_pcb (KiCad board)
At the start: 4 copper layers, 84.3 x 50.8 mm, 128 parts, among them J1 USB_B, J2 USB_A, J3 Barrel_Jack_Switch, J4 Micro_SD_Card, J5 Conn_02x05_Odd_Even, J6 Conn_01x04_Male, J7 Conn_Coaxial, J8 Conn_Coaxial, J9 Conn_Coaxial, Q1 NMOS 2A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

Commit message: Add files via upload
Connections:
- net Net-(C9-Pad1) renamed VCAPL
- net Net-(C9-Pad2) renamed VCAPH
- net Net-(Q1-Pad1) renamed GATE_DRV
- U3 pad 10: Net-(U3-Pad10) -> +3V3
- U3 pad 9: Net-(U3-Pad9) -> +3V3
Routing:
- net +3V3: track 69.8 -> 73.4 mm
