File: PrecisionTimer_RevG.1/PCB Design Files/PrecisionTimer_RevG-1.sch (KiCad schematic (older format))
At the start: 70 parts, among them J1 USB_B, J2 USB_A, J3 Barrel_Jack_Switch, J4 Micro_SD_Card, J5 Conn_02x05_Odd_Even, J6 Conn_01x04_Male, J7 Conn_Coaxial, J8 Conn_Coaxial, J9 Conn_Coaxial, U1 TDC7200PW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

Commit message: Add files via upload
Connections:
- net +3V3: now also U3.10 (RESET#), U3.9 (PROG#)
Changed lines of the file:
@@
-$EndComp
-$Comp
-L power:+3V3 #PWR?
-U 1 1 60400833
-P 6800 4050
-AR Path="/5F82CBFD/60400833" Ref="#PWR?"  Part="1"
-AR Path="/60400833" Ref="#PWR099"  Part="1"
-F 0 "#PWR099" H 6800 3900 50  0001 C CNN
-F 1 "+3V3" H 6815 4223 50  0000 C CNN
-F 2 "" H 6800 4050 50  0001 C CNN
-F 3 "" H 6800 4050 50  0001 C CNN
-	1    6800 4050
-	-1   0    0    1
 $EndComp
 $Comp
@@
 Wire Notes Line
 	2700 1300 2700 4300
+$Comp
+L power:+3V3 #PWR?
+U 1 1 6084C140
+P 6400 4100
+AR Path="/5F82CBFD/6084C140" Ref="#PWR?"  Part="1"
+AR Path="/6084C140" Ref="#PWR?"  Part="1"
+F 0 "#PWR?" H 6400 3950 50  0001 C CNN
+F 1 "+3V3" H 6500 4250 50  0000 C CNN
+F 2 "" H 6400 4100 50  0001 C CNN
+F 3 "" H 6400 4100 50  0001 C CNN
+	1    6400 4100
+	-1   0    0    1
+$EndComp
+Wire Wire Line
+	6400 4050 6400 4100
+Wire Wire Line
+	6400 4100 6500 4100
+Wire Wire Line
+	6800 4100 6800 4050
+Connection ~ 6400 4100
+Wire Wire Line
+	6500 4050 6500 4100
+Connection ~ 6500 4100
+Wire Wire Line
+	6500 4100 6800 4100
 $EndSCHEMATC
